Commit message: feat: complete de urdf to test gazebo and ros_control

File: onedof_description/urdf/onedof.xacro (robot description, xacro)
@@ -1,4 +1,4 @@
 <?xml version="1.0"?>
-<!-- Revolute Manipulator -->
+<!-- just one degree of freedom to test ros_control with gazebo and arduino + dynamixel motor -->
 <robot name="onedof" xmlns:xacro="http://www.ros.org/wiki/xacro">
   <!-- Constants for robot dimensions -->
@@ -25,4 +25,11 @@
   <!-- Base Link -->
   <link name="base_link">
+    <collision>
+      <origin xyz="0 0 0" rpy="0 0 0"/>
+      <geometry>
+	      <!-- <box size="${width} ${width} ${height1}"/> -->
+        <cylinder length = "${height1}" radius="${radius1}" />
+      </geometry>
+    </collision>
     <visual>
       <origin xyz="0 0 0" rpy="0 0 0"/>
@@ -33,4 +40,12 @@
       <material name="orange"/>
     </visual>
+    <inertial>
+      <origin xyz="0 0 0" rpy="0 0 0"/>
+      <mass value="${mass}"/>
+      <inertia
+        ixx = "${mass / 12.0 * (3*radius1*radius1 + height1*height1)}" ixy="0.0" ixz="0.0"
+        iyy = "${mass / 12.0 * (3*radius1*radius1 + height1*height1)}" iyz="0.0"
+        izz="${mass / 2.0 * radius1*radius1}"/>
+    </inertial>
   </link>
   <joint name="joint1" type="continuous">
@@ -40,7 +55,14 @@
     <axis xyz="0 0 1"/>
     <dynamics damping="0.7"/>
+    <dynamics friction="0.3"/>
   </joint>
   <!-- arm Link -->
   <link name="link2">
+    <collision>
+      <origin xyz="0 0 ${length_arm/2-radius1}" rpy="0 0 0"/>
+      <geometry>
+      	<box size="${width} ${length_arm} ${width}"/>
+      </geometry>
+    </collision>
     <visual>
       <origin xyz="0 ${length_arm/2-radius1} 0" rpy="0 0 0"/>
@@ -50,4 +72,12 @@
       <material name="black"/>
     </visual>
+    <inertial>
+      <origin xyz="0 0 ${height2/2 - axel_offset}" rpy="0 0 0"/>
+      <mass value="${mass}"/>
+      <inertia
+        ixx="${mass / 12.0 * (width*width + width*width)}" ixy="0.0" ixz="0.0"
+        iyy="${mass / 12.0 * (length_arm*length_arm + width*width)}" iyz="0.0"
+        izz="${mass / 12.0 * (length_arm*length_arm + width*width)}"/>
+    </inertial>
   </link>
 </robot>

Commit message: feat: modelo urdf, control y gazebo packages for onedof demo

File: onedof_description/urdf/onedof.xacro (robot description, xacro)
@@ -13,5 +13,5 @@
   <xacro:property name="axel_offset" value="0.1" /> <!-- Space btw top of beam and the each joint -->
   <!-- Import all Gazebo-customization elements, including Gazebo colors -->
-  <!-- <xacro:include filename="$(find rrbot_description)/urdf/rrbot.gazebo" /> -->
+  <xacro:include filename="$(find onedof_description)/urdf/onedof.gazebo" />
   <!-- Import Rviz colors -->
   <xacro:include filename="$(find onedof_description)/urdf/materials.xacro" />
@@ -81,3 +81,14 @@
     </inertial>
   </link>
+  <!-- Gazebo element to include the actuator -->
+  <transmission name="tran1">
+    <type>transmission_interface/SimpleTransmission</type>
+    <joint name="joint1">
+      <hardwareInterface>hardware_interface/EffortJointInterface</hardwareInterface>
+    </joint>
+    <actuator name="motor1">
+      <hardwareInterface>hardware_interface/EffortJointInterface</hardwareInterface>
+      <mechanicalReduction>1</mechanicalReduction>
+    </actuator>
+  </transmission>
 </robot>

Commit message: feat: onedof robot  working

File: onedof_description/urdf/onedof.xacro (robot description, xacro)
@@ -54,5 +54,5 @@
     <origin xyz="0 0 ${height1/2+axel_offset}" rpy="0 0 0"/>
     <axis xyz="0 0 1"/>
-    <dynamics damping="0.7"/>
+    <dynamics damping="0.0"/>
     <dynamics friction="0.3"/>
   </joint>
@@ -60,5 +60,5 @@
   <link name="link2">
     <collision>
-      <origin xyz="0 0 ${length_arm/2-radius1}" rpy="0 0 0"/>
+      <origin xyz="0 ${length_arm/2-radius1} 0" rpy="0 0 0"/>
       <geometry>
       	<box size="${width} ${length_arm} ${width}"/>
